File: POWER_DISTRIBUTION/POWER DISTRIBUTIO BOARD_BALLOON/PDB_EXT_CONNECTORS.kicad_sch (KiCad schematic)
At the start: 84 parts, among them J1 Conn_01x02_Socket, J10 Conn_01x02, J11 Conn_01x02, J12 43650-0211, J13 43650-0211, J14 43650-0211, J15 43650-0211, J16 43650-0211, J17 43650-0312, J18 43650-0312, J19 43650-0312, J2 Conn_01x02_Socket, J20 43650-0312, J21 43650-0211, J22 43650-0211, J23 43650-0211, J24 BM12B-GHS-TBT_LF__SN_, J25 43650-0211, J26 BM12B-GHS-TBT_LF__SN_, J27 43650-0211, J28 Conn_01x06, J3 XT90PW-F, J30 Conn_01x02, J31 Conn_01x02, J32 Conn_01x04, J33 Conn_01x02, J34 Conn_01x02, J35 Conn_01x03, J36 Conn_01x03, J4 XT90PW-F, J5 Conn_01x02_Socket, J6 XT90PW-F, J7 XT90PW-F, J8 Conn_01x02, J9 Conn_01x02, U4 178.6165.0002, U5 178.6165.0002, U7 USBLC6-2SC6

Commit message: layout yweaks
Parts:
- J10, J30, J31, J8: footprint Connector_JST:JST_PH_B2B-PH-K_1x02_P2.00mm_Vertical -> Connector_JST:JST_PH_S2B-PH-K_1x02_P2.00mm_Horizontal
- J28: footprint Connector_JST:JST_PH_B6B-PH-K_1x06_P2.00mm_Vertical -> Connector_JST:JST_PH_S5B-PH-SM4-TB_1x05-1MP_P2.00mm_Horizontal
- J32: footprint Connector_JST:JST_PH_B4B-PH-K_1x04_P2.00mm_Vertical -> Connector_JST:JST_PH_S2B-PH-K_1x02_P2.00mm_Horizontal
Changed lines of the file:
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@@
 			)
 		)
-		(property "Footprint" "Connector_JST:JST_PH_B2B-PH-K_1x02_P2.00mm_Vertical"
+		(property "Footprint" "Connector_JST:JST_PH_S2B-PH-K_1x02_P2.00mm_Horizontal"
 			(at 44.45 87.63 0)
 			(effects
@@
 			)
 		)
-		(property "Footprint" "Connector_JST:JST_PH_B2B-PH-K_1x02_P2.00mm_Vertical"
+		(property "Footprint" "Connector_JST:JST_PH_S2B-PH-K_1x02_P2.00mm_Horizontal"
 			(at 111.76 60.96 0)
 			(effects
@@
 			)
 		)
-		(property "Footprint" "Connector_JST:JST_PH_B2B-PH-K_1x02_P2.00mm_Vertical"
+		(property "Footprint" "Connector_JST:JST_PH_S2B-PH-K_1x02_P2.00mm_Horizontal"
 			(at 41.91 123.19 0)
 			(effects
@@
 			)
 		)
-		(property "Footprint" "Connector_JST:JST_PH_B2B-PH-K_1x02_P2.00mm_Vertical"
+		(property "Footprint" "Connector_JST:JST_PH_S2B-PH-K_1x02_P2.00mm_Horizontal"
 			(at 182.88 59.69 0)
 			(effects
@@
 			)
 		)
-		(property "Footprint" "Connector_JST:JST_PH_B4B-PH-K_1x04_P2.00mm_Vertical"
+		(property "Footprint" "Connector_JST:JST_PH_S2B-PH-K_1x02_P2.00mm_Horizontal"
 			(at 138.43 110.49 0)
 			(effects
@@
 			)
 		)
-		(property "Footprint" "Connector_JST:JST_PH_B6B-PH-K_1x06_P2.00mm_Vertical"
+		(property "Footprint" "Connector_JST:JST_PH_S5B-PH-SM4-TB_1x05-1MP_P2.00mm_Horizontal"
 			(at 259.08 46.99 0)
 			(effects
