File: POWER_DISTRIBUTION/POWER DISTRIBUTIO BOARD_BALLOON/PDB_EXT_CONNECTORS.kicad_sch (KiCad schematic)
At the start: 84 parts, among them J1 Conn_01x02_Socket, J10 Conn_01x02, J11 Conn_01x02, J12 43650-0211, J13 43650-0211, J14 43650-0211, J15 43650-0211, J16 43650-0211, J17 43650-0312, J18 43650-0312, J19 43650-0312, J2 Conn_01x02_Socket, J20 43650-0312, J21 43650-0211, J22 43650-0211, J23 43650-0211, J24 BM12B-GHS-TBT_LF__SN_, J25 43650-0211, J26 BM12B-GHS-TBT_LF__SN_, J27 43650-0211, J28 Conn_01x06, J3 XT90PW-F, J30 Conn_01x02, J31 Conn_01x02, J32 Conn_01x04, J33 Conn_01x02, J34 Conn_01x02, J35 Conn_01x03, J36 Conn_01x03, J4 XT90PW-F, J5 Conn_01x02_Socket, J6 XT90PW-F, J7 XT90PW-F, J8 Conn_01x02, J9 Conn_01x02, U4 178.6165.0002, U5 178.6165.0002, U7 USBLC6-2SC6

Commit message: LAYOUT CHANGES TO
Parts:
- removed TP27: S2761-46R, TestPoint:TestPoint_Pad_2.0x2.0mm, symbol samac_sys:S2761-46R
- added TP25, TP26: TestPoint, TestPoint:TestPoint_Pad_1.5x1.5mm, symbol Connector:TestPoint
- J32: footprint Connector_JST:JST_PH_S2B-PH-K_1x02_P2.00mm_Horizontal -> Connector_JST:JST_PH_B6B-PH-K_1x06_P2.00mm_Vertical
- J35, J36: footprint Connector_JST:JST_PH_B3B-PH-K_1x03_P2.00mm_Vertical -> Connector_JST:JST_PH_S3B-PH-K_1x03_P2.00mm_Horizontal
- J9: footprint Connector_JST:JST_PH_B2B-PH-K_1x02_P2.00mm_Vertical -> Connector_JST:JST_PH_S2B-PH-K_1x02_P2.00mm_Horizontal
Connections:
- net +5V0: now also J30.2 (Pin_2), J31.2 (Pin_2), J9.2 (Pin_2), TP25.1; no longer J30.1 (Pin_1), J31.1 (Pin_1), J9.1 (Pin_1)
- net GND: now also J30.1 (Pin_1), J31.1 (Pin_1), J9.1 (Pin_1), TP26.1; no longer J30.2 (Pin_2), J31.2 (Pin_2), J9.2 (Pin_2)
Other:
- moved on the sheet: D10, D12, D13, J30
