File: POWER_DISTRIBUTION/POWER DISTRIBUTIO BOARD_BALLOON/POWER DISTRIBUTIONB BOARD.kicad_pcb (KiCad board)
At the start: 4 copper layers, 74.5 x 55 mm, 102 parts, among them IC3 TPS1HB08BQPWPRQ1, IC4 TPS1HB08BQPWPRQ1, IC8 INA232AIDDFR, IC9 TCAN1044VDDFR, J10 Conn_01x02, J11 Conn_01x02, J28 Conn_01x06, J29 Conn_01x02, J30 Conn_01x02, J31 Conn_01x02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

Commit message: edited the pcb
Parts:
- moved R60 4.18 mm to (175.2, 84.5), turned to 0 degrees
- moved D12 2.90 mm to (175.7, 81.5), turned to 180 degrees
Routing:
- net VTX_EN: track 11.7 -> 52.9 mm
- net HEATER_EN: track 0.00 -> 23.1 mm
- net +3V3: track 18.4 -> 29.8 mm, vias 21 -> 19
- net GND: track 60.8 -> 70.7 mm, vias 70 -> 83
- net VBAT_Fused: track 0.00 -> 7.94 mm
- net VBAT_Fused_OUT: track 0.00 -> 4.37 mm, vias 0 -> 2
- net I2C2_SDA: track 52.9 -> 55.1 mm
- net Net-(Q3-GATE): track 15.1 -> 16.5 mm
- net onewire2: track 29.1 -> 29.9 mm
- net Net-(D12-K): track 7.97 -> 8.75 mm
- net PGM_RX: track 18.7 -> 19.4 mm
- net Net-(C53-Pad1): vias 3 -> 2

Commit message: pcb edits
Routing:
- net Net-(D1-A): track 13.0 -> 14.9 mm
Changed lines of the file:
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@@
+	)
+	(segment
+		(start 183.374 86.124)
+		(end 183.374 87.2)
+		(width 0.254)
+		(layer "F.Cu")
+		(net 11)
+	)
+	(segment
+		(start 182.9405 86)
+		(end 183.25 86)
+		(width 0.254)
+		(layer "F.Cu")
+		(net 11)
 	)
 	(segment
@@
 		(start 178.917543 88.7875)
 		(end 179.512 88.7875)
+		(width 0.254)
+		(layer "F.Cu")
+		(net 11)
+	)
+	(segment
+		(start 183.25 86)
+		(end 183.374 86.124)
 		(width 0.254)
 		(layer "F.Cu")
@@
 	)
 	(via
-		(at 183.374 87.2)
+		(at 182.9405 86)
 		(size 0.61)
 		(drill 0.3)
@@
 	)
 	(segment
-		(start 183.374 87.2)
+		(start 182.05 86.7)
 		(end 182.05 87.2)
+		(width 0.254)
+		(layer "B.Cu")
+		(net 11)
+	)
+	(segment
+		(start 182.9405 86)
+		(end 182.75 86)
 		(width 0.254)
 		(layer "B.Cu")
@@
 		(start 182.05 87.2)
 		(end 181.359917 87.890083)
+		(width 0.254)
+		(layer "B.Cu")
+		(net 11)
+	)
+	(segment
+		(start 182.75 86)
+		(end 182.05 86.7)
 		(width 0.254)
 		(layer "B.Cu")
@@
 			(pts
 				(xy 179.2 98.45) (xy 179.2 97.05) (xy 179.8 96.25) (xy 179.8 90.05) (xy 178.2 90.05) (xy 178.079992 90.05)
-				(xy 177 90.949993) (xy 177 98.45) (xy 178.4 98.45) (xy 178.4 98.45)
+				(xy 177 90.949993) (xy 177 98.45) (xy 178.4 98.45)
 			)
 		)

Commit message: edited pcb
Parts:
- removed R49, R51, R60, R61: 4.7k, Resistor_SMD:R_0603_1608Metric
- D8: moved to B.Cu
- moved R59 14.3 mm to (135.2, 107.8), turned to 90 degrees
- moved D11 13.9 mm to (146.8, 111.5), turned to 0 degrees
- moved J29 13.7 mm to (140.8, 110.2), turned to 90 degrees
- moved R58 12.3 mm to (137.2, 110.5), turned to 90 degrees
- moved C51 10.6 mm to (129.2, 101.9)
- moved C52 10.6 mm to (126.7, 108.2)
- moved IC9 10.6 mm to (129.4, 106.9)
- moved C53 10.1 mm to (137.2, 107.0), turned to 90 degrees
- moved J28 10.0 mm to (117.5, 122.2)
- moved R54 10.0 mm to (123.0, 115.0)
- moved R55 10.0 mm to (125.0, 117.8)
- moved TP30 10.0 mm to (129.2, 117.2)
- moved U6 9.99 mm to (123.5, 102.3)
- moved C48 9.78 mm to (116.5, 114.2)
- moved C49 9.78 mm to (120.0, 114.2)
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Connections:
- D10 pad 3: Net-(D10-K) -> +5V0
- D12 pad 3: Net-(D12-K) -> +5V0
- D13 pad 3: Net-(D13-K) -> +5V0
- D8 pad 3: /EXTERNAL CONNECTORS/BAS_IN -> VBAT+
- J11 pad 2: /EXTERNAL CONNECTORS/BAS_IN -> GND
- J30 pad 2: Net-(D12-K) -> GND
- J31 pad 2: Net-(D13-K) -> GND
- J9 pad 2: Net-(D10-K) -> GND
- TP11 pad 1: /EXTERNAL CONNECTORS/BAS_IN -> GND
Routing:
- net VTX_EN: track 52.9 -> 111.4 mm, vias 1 -> 2
- net HEATER_EN: track 23.1 -> 56.4 mm, vias 0 -> 2
- net CAN+: track 6.45 -> 19.8 mm
- net CAN-: track 5.75 -> 18.5 mm
- net onewire1: track 22.2 -> 34.2 mm, vias 0 -> 1
- net I2C2_SDA: track 55.1 -> 64.6 mm
- net I2C2_SDL: track 48.7 -> 57.8 mm
- net Net-(D10-K): track 8.95 -> 0.00 mm
- net Net-(D12-K): track 8.75 -> 0.00 mm
- net Net-(Q3-GATE): track 16.5 -> 24.8 mm, vias 2 -> 4
- net Net-(D13-K): track 7.82 -> 0.00 mm
- net onewire2: track 29.9 -> 37.6 mm
- net Net-(C53-Pad1): track 4.80 -> 10.3 mm
- net PGM_RX: track 19.4 -> 24.9 mm
- net GND: track 70.7 -> 66.5 mm, vias 83 -> 79
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- added copper zone on B.Cu, net +5V0
- removed copper zone on F.Cu, net /EXTERNAL CONNECTORS/BAS_IN
Other:
- board size 74.5 x 55 mm -> 94.5 x 55 mm
- board text added: "6PINOUT"
- board text added: "CAN"
- board text added: "ONE WIRE"
- board text added: "ONE WIRE2"
- board text added: "PGM"

Commit message: ADD BOARD SCREENSHOT, FIX TRACE
Other:
- board size 94.5 x 55 mm -> 84.5 x 55 mm
- board text added: "PDB REV1.0 DESIGNED BY: SAI WAI PHYO 9V1WP ALVIN TAN YEAN LIANG NUS SATELLITE RESEARCH CENTRE"
Changed lines of the file:
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@@
 			(at 0.05 0.75 0)
 			(layer "F.SilkS")
+			(hide yes)
 			(effects
 				(font
@@
 			(at -3.8006 -1.6852 0)
 			(layer "F.SilkS")
+			(hide yes)
 			(effects
 				(font
@@
 		(tags "Power Supply")
 		(property "Reference" "PS4"
-			(at 0 -2.8 0)
+			(at -3.5 0.2 90)
 			(layer "F.SilkS")
 			(effects
@@
 			(at 5.25 -2.9 0)
 			(layer "F.SilkS")
+			(hide yes)
 			(effects
 				(font
@@
 	)
 	(gr_line
-		(start 198.5 126.5)
-		(end 104 126.5)
+		(start 198.5 127)
+		(end 114 127)
 		(stroke
 			(width 0.05)
@@
 		)
 	)
+	(gr_text "PDB REV1.0\nDESIGNED BY: \nSAI WAI PHYO 9V1WP\nALVIN TAN YEAN LIANG\nNUS SATELLITE RESEARCH CENTRE"
+		(at 140.5 102.75 90)
+		(layer "F.SilkS")
+		(effects
+			(font
+				(size 0.8 0.8)
+				(thickness 0.2)
+				(bold yes)
+			)
+			(justify left bottom)
+		)
+	)
 	(gr_text "+"
 		(at 170.515 73.75 0)
@@
 		(layer "F.Fab")
 		(pts
-			(xy 124 72) (xy 199 72)
+			(xy 114 72) (xy 199 72)
 		)
 		(height -5.75)
@@
 			(keep_text_aligned yes)
 		)
-		(gr_text "75"
-			(at 161.5 65.1 0)
+		(gr_text "85"
+			(at 156.5 65.1 0)
 			(layer "F.Fab")
 			(effects
@@
 	)
 	(segment
-		(start 139.437499 110.25)
-		(end 140.75 110.25)
-		(width 0.1524)
-		(layer "B.Cu")
-		(net 16)
-	)
-	(segment
-		(start 129.3208 108.389848)
-		(end 129.3208 108.973248)
-		(width 0.1524)
-		(layer "B.Cu")
-		(net 16)
-	)
-	(segment
-		(start 129.844556 109.278028)
-		(end 138.465527 109.278028)
+		(start 129.5 109.5)
+		(end 138.687499 109.5)
 		(width 0.1524)
 		(layer "B.Cu")
@@
 	)
 	(segment
-		(start 129.3208 108.973248)
-		(end 129.539776 108.973248)
+		(start 138.687499 109.5)
+		(end 139.437499 110.25)
 		(width 0.1524)
 		(layer "B.Cu")
@@
 	)
 	(segment
-		(start 129.1 108.169048)
-		(end 129.3208 108.389848)
+		(start 139.437499 110.25)
+		(end 140.75 110.25)
 		(width 0.1524)
 		(layer "B.Cu")
@@
 	)
 	(segment
-		(start 129.539776 108.973248)
-		(end 129.844556 109.278028)
+		(start 129.1 109.1)
+		(end 129.5 109.5)
 		(width 0.1524)
 		(layer "B.Cu")
@@
 	)
 	(segment
-		(start 138.465527 109.278028)
-		(end 139.437499 110.25)
+		(start 129.1 108.169048)
+		(end 129.1 109.1)
 		(width 0.1524)
 		(layer "B.Cu")
@@
 	)
 	(segment
-		(start 129.9708 108.973248)
-		(end 138.714251 108.973248)
+		(start 129.9696 109.2196)
+		(end 136.653232 109.2196)
 		(width 0.1524)
 		(layer "B.Cu")
@@
 	)
 	(segment
-		(start 129.9708 108.608795)
-		(end 129.9708 108.973248)
+		(start 136.653232 109.2196)
+		(end 136.802032 109.0708)
+		(width 0.1524)
+		(layer "B.Cu")
+		(net 17)
+	)
+	(segment
+		(start 139.437499 108.25)
+		(end 140.75 108.25)
 		(width 0.1524)
 		(layer "B.Cu")
@@
 	)
 	(segment
-		(start 138.714251 108.973248)
+		(start 138.467899 109.2196)
 		(end 139.437499 108.25)
 		(width 0.1524)
@@
 	)
 	(segment
+		(start 137.846768 109.2196)
+		(end 138.467899 109.2196)
+		(width 0.1524)
+		(layer "B.Cu")
+		(net 17)
+	)
+	(segment
+		(start 129.75 109)
+		(end 129.9696 109.2196)
+		(width 0.1524)
+		(layer "B.Cu")
+		(net 17)
+	)
+	(segment
 		(start 129.75 108.169048)
 		(end 129.75 108.544048)
@@
 	)
 	(segment
-		(start 129.75 108.387995)
-		(end 129.9708 108.608795)
+		(start 136.802032 109.0708)
+		(end 137.697968 109.0708)
 		(width 0.1524)
 		(layer "B.Cu")
@@
 	)
 	(segment
-		(start 139.437499 108.25)
-		(end 140.75 108.25)
+		(start 137.697968 109.0708)
+		(end 137.846768 109.2196)
 		(width 0.1524)
 		(layer "B.Cu")
@@
 	(segment
 		(start 129.75 108.169048)
-		(end 129.75 108.387995)
+		(end 129.75 109)
 		(width 0.1524)
 		(layer "B.Cu")

Commit message: layout yweaks
Parts:
- FB1: footprint SamacSys_COMMS:BEADC2012X105N -> SamacSys_Parts:BEADC2012X105N
- J10, J29, J30, J31, J8: footprint Connector_JST:JST_PH_B2B-PH-K_1x02_P2.00mm_Vertical -> Connector_JST:JST_PH_S2B-PH-K_1x02_P2.00mm_Horizontal
- J28: footprint Connector_JST:JST_PH_B6B-PH-K_1x06_P2.00mm_Vertical -> Connector_JST:JST_PH_S5B-PH-SM4-TB_1x05-1MP_P2.00mm_Horizontal
- J32: footprint Connector_JST:JST_PH_B4B-PH-K_1x04_P2.00mm_Vertical -> Connector_JST:JST_PH_S2B-PH-K_1x02_P2.00mm_Horizontal
- PS4: footprint SamacSys_COMMS:SOT95P280X145-5N -> SamacSys_Parts:SOT95P280X145-5N
- Q3, Q4: footprint SamacSys_COMMS:SOIC127P600X175-8N -> SamacSys_Parts:SOIC127P600X175-8N
- R14, R7: value 13.3k -> 82K
- moved TP30 49.7 mm to (140.3, 68.8)
- moved TP27 6.77 mm to (162.0, 81.2)
- moved PS4 5.48 mm to (152.0, 86.0)
- moved C14 5.48 mm to (152.8, 81.0)
- moved C16 5.48 mm to (152.8, 83.0)
- moved C20 5.48 mm to (145.5, 87.3)
- moved C54 5.48 mm to (147.8, 87.3)
- moved FB1 5.48 mm to (144.5, 83.5)
- moved TP29 4.04 mm to (196.5, 89.0)
- moved C47 2.85 mm to (165.3, 110.6), turned to 0 degrees
- moved IC8 2.83 mm to (164.3, 113.0), turned to 180 degrees
- moved D13 2.70 mm to (159.2, 83.5), turned to -90 degrees
- moved J8 2.60 mm to (192.2, 91.8)
- moved J10 2.55 mm to (192.2, 102.5)
- moved R57 1.27 mm to (143.8, 96.0)
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Routing:
- net GND: track 66.5 -> 51.3 mm, vias 79 -> 110
- net I2C2_SDA: track 64.6 -> 56.6 mm, vias 2 -> 5
- net +3V3: track 32.2 -> 24.8 mm
- net +5V0: track 2.79 -> 8.18 mm, vias 9 -> 6
- net I2C2_SDL: track 57.8 -> 53.1 mm, vias 0 -> 3
- net 12V_BUS2: track 8.21 -> 3.47 mm
- net VBAT_Fused: track 7.94 -> 4.83 mm
- net Net-(IC3-LATCH): track 9.26 -> 10.7 mm
- net Net-(IC3-SNS): track 6.18 -> 7.63 mm
- net HEATER_EN: track 56.4 -> 55.0 mm
- net 12V_BUS1: track 4.29 -> 3.05 mm, vias 0 -> 1
- net Net-(IC3-EN): track 5.79 -> 6.99 mm
- net VBAT_Fused_OUT: track 4.37 -> 5.55 mm
- net Net-(D2-A): track 14.0 -> 12.9 mm
- net VTX_EN: track 111.4 -> 110.3 mm
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Other:
- board text added: "PDB REV1.0 DESIGNED BY: SAI WAI PHYO 9V1WP ALVIN TAN YEAN LIANG NUS STAR 2026"
- board text removed: "PDB REV1.0 DESIGNED BY: SAI WAI PHYO 9V1WP ALVIN TAN YEAN LIANG NUS SATELLITE RESEARCH CENTRE"

Commit message: LAYOUT CHANGES TO
Parts:
- added TP25: TestPoint, TestPoint:TestPoint_Pad_1.5x1.5mm, F.Cu at (156.5, 66.2)
- added TP26: TestPoint, TestPoint:TestPoint_Pad_1.5x1.5mm, B.Cu at (184.5, 75.5)
- J32: footprint Connector_JST:JST_PH_S2B-PH-K_1x02_P2.00mm_Horizontal -> Connector_JST:JST_PH_B6B-PH-K_1x06_P2.00mm_Vertical
- J35, J36: footprint Connector_JST:JST_PH_B3B-PH-K_1x03_P2.00mm_Vertical -> Connector_JST:JST_PH_S3B-PH-K_1x03_P2.00mm_Horizontal
- J9: footprint Connector_JST:JST_PH_B2B-PH-K_1x02_P2.00mm_Vertical -> Connector_JST:JST_PH_S2B-PH-K_1x02_P2.00mm_Horizontal
- TP27: moved to B.Cu
- moved J35 28.6 mm to (156.5, 79.2), turned to 180 degrees
- moved J36 21.0 mm to (136.5, 79.2), turned to 180 degrees
- moved FB1 16.7 mm to (154.9, 96.6), turned to -90 degrees
- moved J28 14.9 mm to (124.4, 135.3)
- moved TP30 12.0 mm to (152.0, 66.2)
- moved C20 10.7 mm to (152.1, 95.7), turned to 180 degrees
- moved J9 9.73 mm to (172.5, 80.5), turned to 180 degrees
- moved J30 9.26 mm to (180.5, 80.5), turned to 180 degrees
- moved J31 9.18 mm to (164.5, 80.5), turned to 180 degrees
- moved D13 8.96 mm to (163.8, 75.8), turned to 180 degrees
- moved D10 8.91 mm to (171.2, 75.5), turned to 180 degrees
- moved D12 8.53 mm to (179.6, 75.8)
- moved C54 7.79 mm to (152.1, 93.7), turned to 180 degrees
- moved C14 7.67 mm to (151.5, 88.6), turned to -90 degrees
- moved TP27 7.27 mm to (157.2, 75.8), turned to 0 degrees
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Connections:
- J30 pad 1: +5V0 -> GND
- J30 pad 2: GND -> +5V0
- J31 pad 1: +5V0 -> GND
- J31 pad 2: GND -> +5V0
- J9 pad 1: +5V0 -> GND
- J9 pad 2: GND -> +5V0
Routing:
- net onewire2: track 37.6 -> 21.6 mm
- net Net-(IC3-LATCH): track 10.7 -> 4.12 mm
- net +5V0: track 8.18 -> 14.1 mm
- net +3V3: track 24.8 -> 20.1 mm
- net Net-(R62-Pad1): track 3.92 -> 8.38 mm
- net Net-(IC3-SNS): track 7.63 -> 4.21 mm
- net BOOT: track 21.9 -> 18.6 mm, vias 2 -> 3
- net GND: track 51.3 -> 54.2 mm, vias 110 -> 118
- added copper zone on B.Cu, net +3V3
Other:
- board size 84.5 x 55 mm -> 85 x 55 mm
- board text added: "5V0"
- board text added: "GND"
