File: POWER_DISTRIBUTION/POWER DISTRIBUTIO BOARD_BALLOON/PDB_CAN.kicad_sch (KiCad schematic)
At the start: 8 parts, among them IC9 TCAN1044VDDFR, J29 Conn_01x02

Commit message: added some global labels
Connections:
- net CAN_RX_FILT_1 renamed CAN_TX
- net CAN_TX_FILT_1 renamed CAN_RX
Changed lines of the file:
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@@
 		)
 	)
-	(global_label "CAN_RX_FILT_1"
+	(global_label "CAN_TX"
 		(shape input)
 		(at 87.63 38.1 180)
@@
 		)
 		(property "Intersheetrefs" "${INTERSHEET_REFS}"
-			(at 70.6748 38.1 0)
+			(at 77.811 38.1 0)
 			(effects
 				(font
@@
 		)
 	)
-	(global_label "CAN_TX_FILT_1"
+	(global_label "CAN_RX"
 		(shape input)
 		(at 87.63 45.72 180)
@@
 		)
 		(property "Intersheetrefs" "${INTERSHEET_REFS}"
-			(at 70.9772 45.72 0)
+			(at 77.5086 45.72 0)
 			(effects
 				(font

Commit message: revert commit
Parts:
- J29: footprint Connector_JST:JST_PH_B2B-PH-K_1x02_P2.00mm_Vertical -> Connector_JST:JST_PH_S2B-PH-K_1x02_P2.00mm_Horizontal
Changed lines of the file:
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@@
 			)
 		)
-		(property "Footprint" "Connector_JST:JST_PH_B2B-PH-K_1x02_P2.00mm_Vertical"
+		(property "Footprint" "Connector_JST:JST_PH_S2B-PH-K_1x02_P2.00mm_Horizontal"
 			(at 132.08 121.92 0)
 			(effects

Commit message: test
Parts:
- J29: footprint Connector_JST:JST_PH_S2B-PH-K_1x02_P2.00mm_Horizontal -> Connector_JST:JST_PH_B2B-PH-K_1x02_P2.00mm_Vertical
Changed lines of the file:
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@@
 			)
 		)
-		(property "Footprint" "Connector_JST:JST_PH_S2B-PH-K_1x02_P2.00mm_Horizontal"
+		(property "Footprint" "Connector_JST:JST_PH_B2B-PH-K_1x02_P2.00mm_Vertical"
 			(at 132.08 121.92 0)
 			(effects
