File: POWER_DISTRIBUTION/POWER DISTRIBUTIO BOARD_BALLOON/PDB_HIGH_SIDE_LOAD_SWITCHES_12VDC_BUS.kicad_sch (KiCad schematic)
At the start: 20 parts, among them IC3 TPS1HB08BQPWPRQ1, IC4 TPS1HB08BQPWPRQ1

Commit message: POWER BOARD LAYOUT COMPLETE
Connections:
- net 12VDC renamed VBAT+
Changed lines of the file:
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@@
+	(wire
+		(pts
+			(xy 128.27 104.14) (xy 128.27 105.41)
+		)
+		(stroke
+			(width 0)
+			(type default)
+		)
+	)
 	(wire
 		(pts
@@
 	(wire
 		(pts
-			(xy 107.95 105.41) (xy 121.92 105.41)
+			(xy 107.95 105.41) (xy 128.27 105.41)
+		)
+		(stroke
+			(width 0)
+			(type default)
+		)
+	)
+	(wire
+		(pts
+			(xy 245.11 104.14) (xy 245.11 105.41)
 		)
 		(stroke
@@
 	)
 	(symbol
+		(lib_id "power:+BATT")
+		(at 128.27 104.14 0)
+		(unit 1)
+		(exclude_from_sim no)
+		(in_bom yes)
+		(on_board yes)
+		(dnp no)
+		(fields_autoplaced yes)
+		(property "Reference" "#PWR0231"
+			(at 128.27 107.95 0)
+			(effects
+				(font
+					(size 1.27 1.27)
+				)
+				(hide yes)
+			)
+		)
+		(property "Value" "VBAT+"
+			(at 128.27 99.06 0)
+			(effects
+				(font
+					(size 1.27 1.27)
+				)
+			)
+		)
+		(property "Footprint" ""
+			(at 128.27 104.14 0)
+			(effects
+				(font
+					(size 1.27 1.27)
+				)
+				(hide yes)
+			)
+		)
+		(property "Datasheet" ""
+			(at 128.27 104.14 0)
+			(effects
+				(font
+					(size 1.27 1.27)
+				)
+				(hide yes)
+			)
+		)
+		(property "Description" "Power symbol creates a global label with name \"+BATT\""
+			(at 128.27 104.14 0)
+			(effects
+				(font
+					(size 1.27 1.27)
+				)
+				(hide yes)
+			)
+		)
+		(pin "1"
+		)
+		(instances
+			(project "POWER DISTRIBUTIONB BOARD"
+				(path "/6b4fba0a-be05-4717-a711-480ed8a7f3e0/6951cc95-37ef-4a4f-8a3f-a120589363a5/28364470-c987-49cb-a285-9d427e41e45e"
+					(reference "#PWR0231")
+					(unit 1)
+				)
+			)
+		)
+	)
+	(symbol
 		(lib_id "power:GND1")
 		(at 62.23 69.85 180)
@@
 	)
 	(symbol
-		(lib_id "power:+BATT")
-		(at 121.92 105.41 270)
-		(unit 1)
-		(exclude_from_sim no)
-		(in_bom yes)
-		(on_board yes)
-		(dnp no)
-		(property "Reference" "#PWR023"
-			(at 118.11 105.41 0)
-			(effects
-				(font
-					(size 1.27 1.27)
-				)
-				(hide yes)
-			)
-		)
-		(property "Value" "12VDC"
-			(at 126.492 105.918 0)
-			(effects
-				(font
-					(size 1.27 1.27)
-				)
-			)
-		)
-		(property "Footprint" ""
-			(at 121.92 105.41 0)
-			(effects
-				(font
-					(size 1.27 1.27)
-				)
-				(hide yes)
-			)
-		)
-		(property "Datasheet" ""
-			(at 121.92 105.41 0)
-			(effects
-				(font
-					(size 1.27 1.27)
-				)
-				(hide yes)
-			)
-		)
-		(property "Description" "Power symbol creates a global label with name \"+BATT\""
-			(at 121.92 105.41 0)
-			(effects
-				(font
-					(size 1.27 1.27)
-				)
-				(hide yes)
-			)
-		)
-		(pin "1"
-		)
-		(instances
-			(project "POWER DISTRIBUTIONB BOARD"
-				(path "/6b4fba0a-be05-4717-a711-480ed8a7f3e0/6951cc95-37ef-4a4f-8a3f-a120589363a5/28364470-c987-49cb-a285-9d427e41e45e"
-					(reference "#PWR023")
-					(unit 1)
-				)
-			)
-		)
-	)
-	(symbol
 		(lib_id "power:GND1")
 		(at 185.42 69.85 180)
@@
 	(symbol
 		(lib_id "power:+BATT")
-		(at 245.11 105.41 270)
-		(unit 1)
-		(exclude_from_sim no)
-		(in_bom yes)
-		(on_board yes)
-		(dnp no)
-		(property "Reference" "#PWR032"
-			(at 241.3 105.41 0)
-			(effects
-				(font
-					(size 1.27 1.27)
-				)
-				(hide yes)
-			)
-		)
-		(property "Value" "12VDC"
-			(at 249.682 105.918 0)
+		(at 245.11 104.14 0)
+		(unit 1)
+		(exclude_from_sim no)
+		(in_bom yes)
+		(on_board yes)
+		(dnp no)
+		(fields_autoplaced yes)
+		(property "Reference" "#PWR0232"
+			(at 245.11 107.95 0)
+			(effects
+				(font
+					(size 1.27 1.27)
+				)
+				(hide yes)
+			)
+		)
+		(property "Value" "VBAT+"
+			(at 245.11 99.06 0)
 			(effects
 				(font
@@
 		)
 		(property "Footprint" ""
-			(at 245.11 105.41 0)
+			(at 245.11 104.14 0)
 			(effects
 				(font
@@
 		)
 		(property "Datasheet" ""
-			(at 245.11 105.41 0)
+			(at 245.11 104.14 0)
 			(effects
 				(font
@@
 		)
 		(property "Description" "Power symbol creates a global label with name \"+BATT\""
-			(at 245.11 105.41 0)
-			(effects
-				(font
-					(size 1.27 1.27)
-				)
-				(hide yes)
-			)
-		)
-		(pin "1"
-		)
-		(instances
-			(project "POWER DISTRIBUTIONB BOARD"
-				(path "/6b4fba0a-be05-4717-a711-480ed8a7f3e0/6951cc95-37ef-4a4f-8a3f-a120589363a5/28364470-c987-49cb-a285-9d427e41e45e"
-					(reference "#PWR032")
-					(unit 1)
-				)
+			(at 245.11 104.14 0)
+			(effects
+				(font
+					(size 1.27 1.27)
+				)
+				(hide yes)
+			)
+		)
+		(pin "1"
+		)
+		(instances
+			(project "POWER DISTRIBUTIONB BOARD"
+				(path "/6b4fba0a-be05-4717-a711-480ed8a7f3e0/6951cc95-37ef-4a4f-8a3f-a120589363a5/28364470-c987-49cb-a285-9d427e41e45e"
+					(reference "#PWR0232")
+					(unit 1)
+				)

Commit message: added some global labels
Connections:
- net HEATER_EN: now reaches R11.1
Changed lines of the file:
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@@
+		)
+	)
+	(global_label "HEATER_EN"
+		(shape input)
+		(at 189.23 91.44 270)
+		(fields_autoplaced yes)
+		(effects
+			(font
+				(size 1.27 1.27)
+			)
+			(justify right)
+		)
+		(property "Intersheetrefs" "${INTERSHEET_REFS}"
+			(at 189.23 104.827 90)
+			(effects
+				(font
+					(size 1.27 1.27)
+				)
+				(justify right)
+				(hide yes)
+			)
 		)
 	)

Commit message: revert commit
Parts:
- R14, R7: value 13.3k -> 82K
Other:
- note added: "EN pin input voltage low-level->0.8BV high-level-2.0V minimum, so can use logic level of epstein32"
- note added: "HEATER(60C 12V) consumes 1A initially Rlim= Kcl/Icl ~11W max 11/11.1~1ohm Kcl==160A*kohm Iclamp=2A Rlim=160/2=80kOhm"

Commit message: test
Parts:
- R14, R7: value 82K -> 13.3k
Other:
- note removed: "EN pin input voltage low-level->0.8BV high-level-2.0V minimum, so can use logic level of epstein32"
- note removed: "HEATER(60C 12V) consumes 1A initially Rlim= Kcl/Icl ~11W max 11/11.1~1ohm Kcl==160A*kohm Iclamp=2A Rlim=160/2=80kOhm"
