File: POWER_DISTRIBUTION/POWER DISTRIBUTIO BOARD_BALLOON/PDB_LOW_SIDE_FETS.kicad_sch (KiCad schematic)
At the start: 8 parts, among them Q1 IPD047N03LF2SATMA1, Q2 IPD047N03LF2SATMA1

Commit message: POWER BOARD LAYOUT COMPLETE
Parts:
- removed Q1, Q2: IPD047N03LF2SATMA1, SamacSys_Parts:IPD047N03LF2SATMA1, symbol samac_sys:IPD047N03LF2SATMA1
- added Q3, Q4: RSS070N05HZGTB, SOIC127P600X175-8N, symbol SamacSys_Parts:RSS070N05HZGTB
Connections:
- net GND: now also Q3.1 (SOURCE_1), Q3.2 (SOURCE_2), Q3.3 (SOURCE_3), Q4.1 (SOURCE_1), Q4.2 (SOURCE_2), Q4.3 (SOURCE_3)
- net PYR_1: now also Q4.5 (DRAIN_1), Q4.6 (DRAIN_2), Q4.7 (DRAIN_3), Q4.8 (DRAIN_4)
- net PYR_2: now also Q3.5 (DRAIN_1), Q3.6 (DRAIN_2), Q3.7 (DRAIN_3), Q3.8 (DRAIN_4)
- net at D6.2, R45.1: now also Q3.4 (GATE)
- net at D5.2, R43.1: now also Q4.4 (GATE)
Other:
- moved on the sheet: D6

Commit message: almost finished wiring
btw for the i2c bus idk if it was meant to be SCL instead of SDL , there is alr an SDA line but i assume so
Parts:
- Q3, Q4: footprint SOIC127P600X175-8N -> SamacSys_COMMS:SOIC127P600X175-8N
Changed lines of the file:
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@@
 			)
 		)
-		(property "Footprint" "SOIC127P600X175-8N"
+		(property "Footprint" "SamacSys_COMMS:SOIC127P600X175-8N"
 			(at 101.6 68.58 0)
 			(effects
@@
 			)
 		)
-		(property "Footprint" "SOIC127P600X175-8N"
+		(property "Footprint" "SamacSys_COMMS:SOIC127P600X175-8N"
 			(at 186.69 68.58 0)
 			(effects

Commit message: revert commit
Parts:
- Q3, Q4: footprint SamacSys_COMMS:SOIC127P600X175-8N -> SamacSys_Parts:SOIC127P600X175-8N
Changed lines of the file:
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@@
 			)
 		)
-		(property "Footprint" "SamacSys_COMMS:SOIC127P600X175-8N"
+		(property "Footprint" "SamacSys_Parts:SOIC127P600X175-8N"
 			(at 101.6 68.58 0)
 			(effects
@@
 			)
 		)
-		(property "Footprint" "SamacSys_COMMS:SOIC127P600X175-8N"
+		(property "Footprint" "SamacSys_Parts:SOIC127P600X175-8N"
 			(at 186.69 68.58 0)
 			(effects

Commit message: test
Parts:
- Q3, Q4: footprint SamacSys_Parts:SOIC127P600X175-8N -> SamacSys_COMMS:SOIC127P600X175-8N
Changed lines of the file:
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@@
 			)
 		)
-		(property "Footprint" "SamacSys_Parts:SOIC127P600X175-8N"
+		(property "Footprint" "SamacSys_COMMS:SOIC127P600X175-8N"
 			(at 101.6 68.58 0)
 			(effects
@@
 			)
 		)
-		(property "Footprint" "SamacSys_Parts:SOIC127P600X175-8N"
+		(property "Footprint" "SamacSys_COMMS:SOIC127P600X175-8N"
 			(at 186.69 68.58 0)
 			(effects
